File: schematic/WirelessTouchLight.kicad_pcb (KiCad board)
At the start: 2 copper layers, 10 parts, among them J1 Conn_01x04, J2 HLK-PM03, K1 HK4100F-DC3V-SHG, Q1 2N2222, U1 WeMos_mini

Commit message: Update schematic
Parts:
- D1: moved to B.Cu
- J1: footprint Terminal_Blocks:TerminalBlock_bornier-4_P5.08mm -> KF-TerminalBlock:KF235-4P
- moved D1 46.3 mm to (46.4, 59.1), turned to 270 degrees
- moved K1 40.9 mm to (41.3, 55.2)
- moved J1 31.1 mm to (52.7, 79.4), turned to 0 degrees
- moved F1 27.5 mm to (57.8, 59.2), turned to 180 degrees
- moved Q1 25.2 mm to (47.9, 43.4), turned to 270 degrees
- moved R1 9.25 mm to (47.0, 35.6), turned to 90 degrees
- moved C1 8.28 mm to (62.2, 56.5), turned to 270 degrees
- moved J2 0.69 mm to (52.1, 35.0), turned to 90 degrees
- moved R2 0.63 mm to (59.7, 33.7)
Routing:
- net VCC: track 0.00 -> 50.4 mm
- net GND: track 0.00 -> 44.7 mm
- net /Live: track 0.00 -> 38.2 mm
- net Net-(C1-Pad1): track 0.00 -> 28.5 mm
- net /Neutral: track 0.00 -> 26.1 mm
- net Net-(D1-Pad2): track 0.00 -> 25.7 mm
- net /TouchSense: track 0.00 -> 14.1 mm
- net /Output: track 0.00 -> 14.0 mm
- net Net-(R1-Pad2): track 0.00 -> 8.19 mm
- net Net-(F1-Pad2): track 0.00 -> 7.93 mm
- net Net-(Q1-Pad1): track 0.00 -> 4.92 mm
- net Net-(R2-Pad2): track 0.00 -> 3.88 mm
Other:
- board outline added: 25.4 x 61.6 mm
- net class large added: clearance 0.4, trace_width 0.5, via_dia 0.8, via_drill 0.4
- board text added: "L"
- board text added: "N"
- board text added: "O"
- board text added: "S"
- board text added: "WirelessTouchLite V1.0"

Commit message: Change to 470K Resistor
Parts:
- R2: value 120K -> 470K
Changed lines of the file:
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@@
     (solder_mask_min_width 0.25)
     (aux_axis_origin 0 0)
-    (visible_elements 7FFDFFFF)
+    (visible_elements 7FFFFFFF)
     (pcbplotparams
       (layerselection 0x010fc_ffffffff)
@@
       (effects (font (size 1 1) (thickness 0.15)))
     )
-    (fp_text value "470pF 3KV" (at 2.5 3.56 90) (layer F.Fab)
+    (fp_text value "470pF 3KV" (at 2.032 1.651 90) (layer F.SilkS)
       (effects (font (size 1 1) (thickness 0.15)))
     )
@@
       (effects (font (size 1 1) (thickness 0.15)) (justify mirror))
     )
-    (fp_text value 120K (at 0 -1.75 270) (layer B.SilkS)
-      (effects (font (size 1 1) (thickness 0.15)) (justify mirror))
-    )
+    (fp_text value 470K (at 0 -1.75 270) (layer B.SilkS)
+      (effects (font (size 1 1) (thickness 0.15)) (justify mirror))
+    )

Commit message: Change Back to 100K resistor (470 too much noises)
Parts:
- R2: value 470K -> 100K
Changed lines of the file:
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@@
       (effects (font (size 1 1) (thickness 0.15)) (justify mirror))
     )
-    (fp_text value 470K (at 0 -1.75 270) (layer B.SilkS)
+    (fp_text value 100K (at 0 -1.75 270) (layer B.SilkS)
       (effects (font (size 1 1) (thickness 0.15)) (justify mirror))
     )

Commit message: Update schematic/PCB
Parts:
- F1: value Polyfuse -> TRF250-1A
Other:
- board text added: "WirelessTouchLight V1.0"
- board text removed: "WirelessTouchLite V1.0"
Changed lines of the file:
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@@
-(kicad_pcb (version 20171130) (host pcbnew "(5.1.4)-1")
+(kicad_pcb (version 20171130) (host pcbnew "(5.1.5)-3")
   (general
     (thickness 1.6)
@@
   (page A4)
   (layers
-    (0 F.Cu signal)
-    (31 B.Cu signal)
+    (0 F.Cu signal hide)
+    (31 B.Cu signal hide)
     (32 B.Adhes user)
     (33 F.Adhes user)
@@
       (effects (font (size 1 1) (thickness 0.15)))
     )
-    (fp_text value Polyfuse (at 0 8.255) (layer F.Fab)
+    (fp_text value TRF250-1A (at -2.5908 5.969) (layer F.SilkS)
       (effects (font (size 1 1) (thickness 0.15)))
     )
@@
       (effects (font (size 1 1) (thickness 0.15)))
     )
-    (fp_text value HLK-PM03 (at 0 -1 90) (layer F.Fab)
+    (fp_text value HLK-PM03 (at 0 -1 90) (layer F.SilkS)
       (effects (font (size 1 1) (thickness 0.15)))
     )
@@
       (effects (font (size 1 1) (thickness 0.15)))
     )
-    (fp_text value HK4100F-DC3V-SHG (at 6.985 2.54) (layer F.Fab)
+    (fp_text value HK4100F-DC3V-SHG (at 6.35 -2.286) (layer F.SilkS)
       (effects (font (size 1 1) (thickness 0.15)))
     )
@@
     (effects (font (size 1.5 1.5) (thickness 0.3)) (justify mirror))
   )
-  (gr_text "WirelessTouchLite\nV1.0" (at 53.975 32.385 90) (layer B.SilkS)
+  (gr_text "WirelessTouchLight\nV1.0" (at 53.975 32.385 90) (layer B.SilkS)
     (effects (font (size 1.5 1.5) (thickness 0.3)) (justify mirror))
   )
